Commit message: update collision model

File: bullet_test/model/bowl/model_viz.urdf (robot description, URDF)
Before this commit: robot pot, 1 links, 0 joints
Links:
- link nil_link: geometry collision mesh filename=model://bowl/meshes/nil_link_mesh.dae scale=1 1 1

File: bullet_test/model/pot/model_viz.urdf (robot description, URDF)
Before this commit: robot pot, 1 links, 0 joints
Links:
- link nil_link: geometry collision mesh filename=model://pot/meshes/nil_link_mesh.dae scale=1 1 1
